File: blt.brd (EAGLE design)
At the start: 100 x 80 mm, 15 parts, among them IC1 TL074D

Commit message: некоторые новые обновления трансмитера
Parts:
- added C1: 680p, rcl:C1206
- added C2: 220p, rcl:C1206
- added C3: 470p, rcl:C1206
- added C4: (no value), rcl:UD-4X5,8_NICHICON
- added IC2: TL074D, linear:SO14
- added R11, R12, R14: 6k8, rcl:R1206
- added R13: 5k6, rcl:R1206
- added R15, R16: 10k, rcl:R1206
Connections:
- new net N$12: C3.2, IC2.1, R14.1, R15.2
- new net N$13: IC2.2, R15.1, R16.2
- new net N$4: R11.1, R12.2
- new net N$5: C2.1, C3.1, IC2.3, R11.2
- new net N$9: C1.1, R12.1, R13.2
- net +15V: now also IC2.4
- net -15V: now also IC2.11
Changed lines of the file:
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@@
 <element name="JP3" library="pinhead" package="1X03" value="Bal_OUT2" x="55.88" y="11.43"/>
 <element name="JP4" library="pinhead" package="1X03" value="UNBAL_IN" x="44.45" y="5.08"/>
+<element name="IC2" library="linear" package="SO14" value="TL074D" x="6.35" y="-6.35"/>
+<element name="R11" library="rcl" package="R1206" value="6k8" x="2.54" y="-13.97"/>
+<element name="R12" library="rcl" package="R1206" value="6k8" x="2.54" y="-20.32"/>
+<element name="R13" library="rcl" package="R1206" value="5k6" x="2.54" y="-26.67"/>
+<element name="C1" library="rcl" package="C1206" value="680p" x="2.54" y="-33.02"/>
+<element name="C2" library="rcl" package="C1206" value="220p" x="2.54" y="-38.1"/>
+<element name="R14" library="rcl" package="R1206" value="6k8" x="2.54" y="-44.45"/>
+<element name="C3" library="rcl" package="C1206" value="470p" x="2.54" y="-50.8"/>
+<element name="R15" library="rcl" package="R1206" value="10k" x="2.54" y="-57.15"/>
+<element name="R16" library="rcl" package="R1206" value="10k" x="2.54" y="-63.5"/>
+<element name="C4" library="rcl" package="UD-4X5,8_NICHICON" value="" x="-5.08" y="-62.23"/>
 </elements>
 <signals>
@@
 <contactref element="JP1" pad="2"/>
 <contactref element="IC1" pad="4"/>
-<wire x1="53.4" y1="40.64" x2="52.07" y2="49.53" width="0" layer="19" extent="1-1"/>
+<contactref element="IC2" pad="4"/>
+<wire x1="53.4" y1="40.64" x2="52.07" y2="49.53" width="0" layer="19" extent="16-16"/>
+<wire x1="6.35" y1="-8.95" x2="53.4" y2="40.64" width="0" layer="19" extent="1-16"/>
 </signal>
 <signal name="-15V">
 <contactref element="JP1" pad="1"/>
 <contactref element="IC1" pad="11"/>
-<wire x1="48.2" y1="40.64" x2="49.53" y2="49.53" width="0" layer="19" extent="1-1"/>
+<contactref element="IC2" pad="11"/>
+<wire x1="48.2" y1="40.64" x2="49.53" y2="49.53" width="0" layer="19" extent="16-16"/>
+<wire x1="6.35" y1="-3.75" x2="48.2" y2="40.64" width="0" layer="19" extent="1-16"/>
 </signal>
 <signal name="+OUT1">
@@
 <wire x1="58.42" y1="11.43" x2="26.518" y2="46.99" width="0" layer="19" extent="16-16"/>
 </signal>
+<signal name="N$4">
+<contactref element="R12" pad="2"/>
+<contactref element="R11" pad="1"/>
+<wire x1="1.118" y1="-13.97" x2="3.962" y2="-20.32" width="0" layer="19" extent="1-1"/>
+</signal>
+<signal name="N$5">
+<contactref element="R11" pad="2"/>
+<contactref element="IC2" pad="3"/>
+<contactref element="C2" pad="1"/>
+<contactref element="C3" pad="1"/>
+<wire x1="1.14" y1="-38.1" x2="1.14" y2="-50.8" width="0" layer="19" extent="1-1"/>
+<wire x1="3.962" y1="-13.97" x2="1.14" y2="-38.1" width="0" layer="19" extent="1-1"/>
+<wire x1="5.08" y1="-8.95" x2="3.962" y2="-13.97" width="0" layer="19" extent="1-1"/>
+</signal>
+<signal name="N$9">
+<contactref element="R13" pad="2"/>
+<contactref element="R12" pad="1"/>
+<contactref element="C1" pad="1"/>
+<wire x1="3.962" y1="-26.67" x2="1.14" y2="-33.02" width="0" layer="19" extent="1-1"/>
+<wire x1="1.118" y1="-20.32" x2="3.962" y2="-26.67" width="0" layer="19" extent="1-1"/>
+</signal>
+<signal name="N$12">
+<contactref element="IC2" pad="1"/>
+<contactref element="R14" pad="1"/>
+<contactref element="C3" pad="2"/>
+<contactref element="R15" pad="2"/>
+<wire x1="3.94" y1="-50.8" x2="3.962" y2="-57.15" width="0" layer="19" extent="1-1"/>
+<wire x1="1.118" y1="-44.45" x2="3.94" y2="-50.8" width="0" layer="19" extent="1-1"/>
+<wire x1="2.54" y1="-8.95" x2="1.118" y2="-44.45" width="0" layer="19" extent="1-1"/>
+</signal>
+<signal name="N$13">
+<contactref element="IC2" pad="2"/>
+<contactref element="R15" pad="1"/>
+<contactref element="R16" pad="2"/>
+<wire x1="1.118" y1="-57.15" x2="3.962" y2="-63.5" width="0" layer="19" extent="1-1"/>
+<wire x1="3.81" y1="-8.95" x2="1.118" y2="-57.15" width="0" layer="19" extent="1-1"/>
+</signal>
 </signals>

Commit message: temp
Parts:
- C4: value (none) -> 4u
- R14: value 6k8 -> 100
- R16: value 10k -> 20k
Connections:
- new net N$14: C4.-, R13.1
- net AGND: now also C1.2, C2.2, R16.1
Changed lines of the file:
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@@
 <element name="C1" library="rcl" package="C1206" value="680p" x="2.54" y="-33.02"/>
 <element name="C2" library="rcl" package="C1206" value="220p" x="2.54" y="-38.1"/>
-<element name="R14" library="rcl" package="R1206" value="6k8" x="2.54" y="-44.45"/>
+<element name="R14" library="rcl" package="R1206" value="100" x="2.54" y="-44.45"/>
 <element name="C3" library="rcl" package="C1206" value="470p" x="2.54" y="-50.8"/>
 <element name="R15" library="rcl" package="R1206" value="10k" x="2.54" y="-57.15"/>
-<element name="R16" library="rcl" package="R1206" value="10k" x="2.54" y="-63.5"/>
-<element name="C4" library="rcl" package="UD-4X5,8_NICHICON" value="" x="-5.08" y="-62.23"/>
+<element name="R16" library="rcl" package="R1206" value="20k" x="2.54" y="-63.5"/>
+<element name="C4" library="rcl" package="UD-4X5,8_NICHICON" value="4u" x="-5.08" y="-62.23"/>
 </elements>
 <signals>
@@
 <contactref element="JP3" pad="2"/>
 <contactref element="JP4" pad="2"/>
+<contactref element="R16" pad="1"/>
+<contactref element="C1" pad="2"/>
+<contactref element="C2" pad="2"/>
 <wire x1="48.2" y1="41.91" x2="53.4" y2="39.37" width="0" layer="19" extent="16-16"/>
-<wire x1="69.85" y1="11.43" x2="48.2" y2="41.91" width="0" layer="19" extent="16-16"/>
-<wire x1="55.88" y1="11.43" x2="69.85" y2="11.43" width="0" layer="19" extent="1-1"/>
+<wire x1="55.88" y1="11.43" x2="53.4" y2="39.37" width="0" layer="19" extent="16-16"/>
 <wire x1="44.45" y1="5.08" x2="55.88" y2="11.43" width="0" layer="19" extent="1-1"/>
+<wire x1="69.85" y1="11.43" x2="55.88" y2="11.43" width="0" layer="19" extent="1-1"/>
+<wire x1="3.94" y1="-33.02" x2="44.45" y2="5.08" width="0" layer="19" extent="1-1"/>
+<wire x1="3.94" y1="-38.1" x2="3.94" y2="-33.02" width="0" layer="19" extent="1-1"/>
+<wire x1="1.118" y1="-63.5" x2="3.94" y2="-38.1" width="0" layer="19" extent="1-1"/>
 </signal>
 <signal name="+15V">
@@
 <wire x1="3.81" y1="-8.95" x2="1.118" y2="-57.15" width="0" layer="19" extent="1-1"/>
 </signal>
+<signal name="N$14">
+<contactref element="C4" pad="-"/>
+<contactref element="R13" pad="1"/>
+<wire x1="1.118" y1="-26.67" x2="-6.505" y2="-62.23" width="0" layer="19" extent="1-1"/>
+</signal>
 </signals>
