File: blt.sch (EAGLE design)
At the start: 15 parts, among them IC1 TL074D

Commit message: некоторые новые обновления трансмитера
Parts:
- added C1: 680p, rcl:C-EUC1206
- added C2: 220p, rcl:C-EUC1206
- added C3: 470p, rcl:C-EUC1206
- added C4: (no value), rcl:CPOL-EUUD-4X5,8
- added IC2: TL074D, linear:TL074D
- added R11, R12, R14: 6k8, rcl:R-EU_R1206
- added R13: 5k6, rcl:R-EU_R1206
- added R15, R16: 10k, rcl:R-EU_R1206
Connections:
- new net N$12: C3.2, IC2A.OUT, R14.1, R15.2
- new net N$13: IC2A.-IN, R15.1, R16.2
- new net N$4: R11.1, R12.2
- new net N$5: C2.1, C3.1, IC2A.+IN, R11.2
- new net N$9: C1.1, R12.1, R13.2
- net +15V: now also IC2P.V+
- net -15V: now also IC2P.V-
Changed lines of the file:
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@@
 <part name="AGND4" library="supply1" deviceset="AGND" device=""/>
 <part name="AGND5" library="supply1" deviceset="AGND" device=""/>
+<part name="IC2" library="linear" deviceset="TL074" device="D"/>
+<part name="R11" library="rcl" deviceset="R-EU_" device="R1206" value="6k8"/>
+<part name="R12" library="rcl" deviceset="R-EU_" device="R1206" value="6k8"/>
+<part name="R13" library="rcl" deviceset="R-EU_" device="R1206" value="5k6"/>
+<part name="C1" library="rcl" deviceset="C-EU" device="C1206" value="680p"/>
+<part name="C2" library="rcl" deviceset="C-EU" device="C1206" value="220p"/>
+<part name="R14" library="rcl" deviceset="R-EU_" device="R1206" value="6k8"/>
+<part name="C3" library="rcl" deviceset="C-EU" device="C1206" value="470p"/>
+<part name="R15" library="rcl" deviceset="R-EU_" device="R1206" value="10k"/>
+<part name="R16" library="rcl" deviceset="R-EU_" device="R1206" value="10k"/>
+<part name="C4" library="rcl" deviceset="CPOL-EU" device="UD-4X5,8"/>
 </parts>
 <sheets>
@@
 <instance part="AGND4" gate="VR1" x="25.4" y="-33.02"/>
 <instance part="AGND5" gate="VR1" x="-15.24" y="-12.7"/>
+<instance part="IC2" gate="A" x="0" y="-73.66"/>
+<instance part="IC2" gate="B" x="0" y="-139.7"/>
+<instance part="IC2" gate="C" x="0" y="-152.4"/>
+<instance part="IC2" gate="D" x="0" y="-165.1" smashed="yes">
+<attribute name="NAME" x="2.54" y="-161.925" size="1.778" layer="95"/>
+<attribute name="VALUE" x="2.54" y="-170.18" size="1.778" layer="96"/>
+</instance>
+<instance part="IC2" gate="P" x="71.12" y="12.7" rot="R90"/>
+<instance part="R11" gate="G$1" x="-25.4" y="-71.12"/>
+<instance part="R12" gate="G$1" x="-40.64" y="-71.12"/>
+<instance part="R13" gate="G$1" x="-58.42" y="-71.12"/>
+<instance part="C1" gate="G$1" x="-50.8" y="-78.74"/>
+<instance part="C2" gate="G$1" x="-17.78" y="-78.74"/>
+<instance part="R14" gate="G$1" x="22.86" y="-73.66"/>
+<instance part="C3" gate="G$1" x="-7.62" y="-63.5" rot="R90"/>
+<instance part="R15" gate="G$1" x="2.54" y="-83.82"/>
+<instance part="R16" gate="G$1" x="-10.16" y="-93.98" rot="R90"/>
+<instance part="C4" gate="G$1" x="-76.2" y="-71.12" rot="R90"/>
 </instances>
 <busses>
@@
 <wire x1="60.96" y1="27.94" x2="66.04" y2="27.94" width="0.1524" layer="91"/>
 <junction x="66.04" y="27.94"/>
+<pinref part="IC2" gate="P" pin="V+"/>
+<wire x1="63.5" y1="12.7" x2="60.96" y2="12.7" width="0.1524" layer="91"/>
+<wire x1="60.96" y1="12.7" x2="60.96" y2="15.24" width="0.1524" layer="91"/>
+<junction x="60.96" y="15.24"/>
 </segment>
 </net>
@@
 <wire x1="81.28" y1="27.94" x2="73.66" y2="27.94" width="0.1524" layer="91"/>
 <junction x="73.66" y="27.94"/>
+<pinref part="IC2" gate="P" pin="V-"/>
+<wire x1="78.74" y1="12.7" x2="81.28" y2="12.7" width="0.1524" layer="91"/>
+<wire x1="81.28" y1="12.7" x2="81.28" y2="15.24" width="0.1524" layer="91"/>
+<junction x="81.28" y="15.24"/>
 </segment>
 </net>
@@
 </segment>
 </net>
+<net name="N$4" class="0">
+<segment>
+<pinref part="R12" gate="G$1" pin="2"/>
+<pinref part="R11" gate="G$1" pin="1"/>
+<wire x1="-35.56" y1="-71.12" x2="-30.48" y2="-71.12" width="0.1524" layer="91"/>
+</segment>
+</net>
+<net name="N$5" class="0">
+<segment>
+<pinref part="R11" gate="G$1" pin="2"/>
+<pinref part="IC2" gate="A" pin="+IN"/>
+<wire x1="-20.32" y1="-71.12" x2="-17.78" y2="-71.12" width="0.1524" layer="91"/>
+<pinref part="C2" gate="G$1" pin="1"/>
+<wire x1="-17.78" y1="-71.12" x2="-7.62" y2="-71.12" width="0.1524" layer="91"/>
+<wire x1="-17.78" y1="-76.2" x2="-17.78" y2="-71.12" width="0.1524" layer="91"/>
+<junction x="-17.78" y="-71.12"/>
+<pinref part="C3" gate="G$1" pin="1"/>
+<wire x1="-10.16" y1="-63.5" x2="-17.78" y2="-63.5" width="0.1524" layer="91"/>
+<wire x1="-17.78" y1="-63.5" x2="-17.78" y2="-71.12" width="0.1524" layer="91"/>
+</segment>
+</net>
+<net name="N$9" class="0">
+<segment>
+<pinref part="R13" gate="G$1" pin="2"/>
+<pinref part="R12" gate="G$1" pin="1"/>
+<wire x1="-53.34" y1="-71.12" x2="-50.8" y2="-71.12" width="0.1524" layer="91"/>
+<pinref part="C1" gate="G$1" pin="1"/>
+<wire x1="-50.8" y1="-71.12" x2="-45.72" y2="-71.12" width="0.1524" layer="91"/>
+<wire x1="-50.8" y1="-76.2" x2="-50.8" y2="-71.12" width="0.1524" layer="91"/>
+<junction x="-50.8" y="-71.12"/>
+</segment>
+</net>
+<net name="N$12" class="0">
+<segment>
+<pinref part="IC2" gate="A" pin="OUT"/>
+<pinref part="R14" gate="G$1" pin="1"/>
+<wire x1="7.62" y1="-73.66" x2="10.16" y2="-73.66" width="0.1524" layer="91"/>
+<pinref part="C3" gate="G$1" pin="2"/>
+<wire x1="10.16" y1="-73.66" x2="17.78" y2="-73.66" width="0.1524" layer="91"/>
+<wire x1="-2.54" y1="-63.5" x2="10.16" y2="-63.5" width="0.1524" layer="91"/>
+<wire x1="10.16" y1="-63.5" x2="10.16" y2="-73.66" width="0.1524" layer="91"/>
+<junction x="10.16" y="-73.66"/>
+<pinref part="R15" gate="G$1" pin="2"/>
+<wire x1="7.62" y1="-83.82" x2="10.16" y2="-83.82" width="0.1524" layer="91"/>
+<wire x1="10.16" y1="-83.82" x2="10.16" y2="-73.66" width="0.1524" layer="91"/>
+</segment>
+</net>
+<net name="N$13" class="0">
+<segment>
+<pinref part="IC2" gate="A" pin="-IN"/>
+<wire x1="-7.62" y1="-76.2" x2="-10.16" y2="-76.2" width="0.1524" layer="91"/>
+<wire x1="-10.16" y1="-76.2" x2="-10.16" y2="-83.82" width="0.1524" layer="91"/>
+<pinref part="R15" gate="G$1" pin="1"/>
+<wire x1="-10.16" y1="-83.82" x2="-2.54" y2="-83.82" width="0.1524" layer="91"/>
+<pinref part="R16" gate="G$1" pin="2"/>
+<wire x1="-10.16" y1="-88.9" x2="-10.16" y2="-83.82" width="0.1524" layer="91"/>
+<junction x="-10.16" y="-83.82"/>
+</segment>
+</net>

Commit message: temp
Parts:
- C4: value (none) -> 4u
- R14: value 6k8 -> 100
- R16: value 10k -> 20k
Connections:
- new net N$14: C4.-, R13.1
- net AGND: now also C1.2, C2.2, R16.1
Changed lines of the file:
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@@
 <grid distance="0.1" unitdist="inch" unit="inch" style="lines" multiple="1" display="yes" altdistance="0.01" altunitdist="inch" altunit="inch"/>
 <layers>
-<layer number="1" name="Top" color="4" fill="1" visible="yes" active="no"/>
-<layer number="16" name="Bottom" color="1" fill="1" visible="yes" active="no"/>
-<layer number="17" name="Pads" color="2" fill="1" visible="yes" active="no"/>
-<layer number="18" name="Vias" color="2" fill="1" visible="yes" active="no"/>
-<layer number="19" name="Unrouted" color="6" fill="1" visible="yes" active="no"/>
-<layer number="20" name="Dimension" color="15" fill="1" visible="yes" active="no"/>
-<layer number="21" name="tPlace" color="7" fill="1" visible="yes" active="no"/>
-<layer number="22" name="bPlace" color="7" fill="1" visible="yes" active="no"/>
-<layer number="23" name="tOrigins" color="15" fill="1" visible="yes" active="no"/>
-<layer number="24" name="bOrigins" color="15" fill="1" visible="yes" active="no"/>
-<layer number="25" name="tNames" color="7" fill="1" visible="yes" active="no"/>
-<layer number="26" name="bNames" color="7" fill="1" visible="yes" active="no"/>
-<layer number="27" name="tValues" color="7" fill="1" visible="yes" active="no"/>
-<layer number="28" name="bValues" color="7" fill="1" visible="yes" active="no"/>
+<layer number="1" name="Top" color="4" fill="1" visible="no" active="no"/>
+<layer number="16" name="Bottom" color="1" fill="1" visible="no" active="no"/>
+<layer number="17" name="Pads" color="2" fill="1" visible="no" active="no"/>
+<layer number="18" name="Vias" color="2" fill="1" visible="no" active="no"/>
+<layer number="19" name="Unrouted" color="6" fill="1" visible="no" active="no"/>
+<layer number="20" name="Dimension" color="15" fill="1" visible="no" active="no"/>
+<layer number="21" name="tPlace" color="7" fill="1" visible="no" active="no"/>
+<layer number="22" name="bPlace" color="7" fill="1" visible="no" active="no"/>
+<layer number="23" name="tOrigins" color="15" fill="1" visible="no" active="no"/>
+<layer number="24" name="bOrigins" color="15" fill="1" visible="no" active="no"/>
+<layer number="25" name="tNames" color="7" fill="1" visible="no" active="no"/>
+<layer number="26" name="bNames" color="7" fill="1" visible="no" active="no"/>
+<layer number="27" name="tValues" color="7" fill="1" visible="no" active="no"/>
+<layer number="28" name="bValues" color="7" fill="1" visible="no" active="no"/>
 <layer number="29" name="tStop" color="7" fill="3" visible="no" active="no"/>
 <layer number="30" name="bStop" color="7" fill="6" visible="no" active="no"/>
@@
 <layer number="35" name="tGlue" color="7" fill="4" visible="no" active="no"/>
 <layer number="36" name="bGlue" color="7" fill="5" visible="no" active="no"/>
-<layer number="37" name="tTest" color="7" fill="1" visible="yes" active="no"/>
-<layer number="38" name="bTest" color="7" fill="1" visible="yes" active="no"/>
+<layer number="37" name="tTest" color="7" fill="1" visible="no" active="no"/>
+<layer number="38" name="bTest" color="7" fill="1" visible="no" active="no"/>
 <layer number="39" name="tKeepout" color="4" fill="11" visible="no" active="no"/>
 <layer number="40" name="bKeepout" color="1" fill="11" visible="no" active="no"/>
@@
 <layer number="44" name="Drills" color="7" fill="1" visible="no" active="no"/>
 <layer number="45" name="Holes" color="7" fill="1" visible="no" active="no"/>
-<layer number="46" name="Milling" color="3" fill="1" visible="yes" active="no"/>
-<layer number="47" name="Measures" color="7" fill="1" visible="yes" active="no"/>
-<layer number="48" name="Document" color="7" fill="1" visible="yes" active="no"/>
-<layer number="49" name="Reference" color="7" fill="1" visible="yes" active="no"/>
-<layer number="51" name="tDocu" color="7" fill="1" visible="yes" active="no"/>
-<layer number="52" name="bDocu" color="7" fill="1" visible="yes" active="no"/>
+<layer number="46" name="Milling" color="3" fill="1" visible="no" active="no"/>
+<layer number="47" name="Measures" color="7" fill="1" visible="no" active="no"/>
+<layer number="48" name="Document" color="7" fill="1" visible="no" active="no"/>
+<layer number="49" name="Reference" color="7" fill="1" visible="no" active="no"/>
+<layer number="51" name="tDocu" color="7" fill="1" visible="no" active="no"/>
+<layer number="52" name="bDocu" color="7" fill="1" visible="no" active="no"/>
 <layer number="90" name="Modules" color="5" fill="1" visible="yes" active="yes"/>
 <layer number="91" name="Nets" color="2" fill="1" visible="yes" active="yes"/>
@@
 <part name="C1" library="rcl" deviceset="C-EU" device="C1206" value="680p"/>
 <part name="C2" library="rcl" deviceset="C-EU" device="C1206" value="220p"/>
-<part name="R14" library="rcl" deviceset="R-EU_" device="R1206" value="6k8"/>
+<part name="R14" library="rcl" deviceset="R-EU_" device="R1206" value="100"/>
 <part name="C3" library="rcl" deviceset="C-EU" device="C1206" value="470p"/>
 <part name="R15" library="rcl" deviceset="R-EU_" device="R1206" value="10k"/>
-<part name="R16" library="rcl" deviceset="R-EU_" device="R1206" value="10k"/>
-<part name="C4" library="rcl" deviceset="CPOL-EU" device="UD-4X5,8"/>
+<part name="R16" library="rcl" deviceset="R-EU_" device="R1206" value="20k"/>
+<part name="C4" library="rcl" deviceset="CPOL-EU" device="UD-4X5,8" value="4u"/>
+<part name="AGND6" library="supply1" deviceset="AGND" device=""/>
+<part name="AGND7" library="supply1" deviceset="AGND" device=""/>
+<part name="AGND8" library="supply1" deviceset="AGND" device=""/>
 </parts>
 <sheets>
@@
 <instance part="R16" gate="G$1" x="-10.16" y="-93.98" rot="R90"/>
 <instance part="C4" gate="G$1" x="-76.2" y="-71.12" rot="R90"/>
+<instance part="AGND6" gate="VR1" x="-10.16" y="-109.22"/>
+<instance part="AGND7" gate="VR1" x="-17.78" y="-109.22"/>
+<instance part="AGND8" gate="VR1" x="-50.8" y="-109.22"/>
 </instances>
 <busses>
@@
 <wire x1="-15.24" y1="-7.62" x2="-15.24" y2="-10.16" width="0.1524" layer="91"/>
 <label x="-38.1" y="-7.62" size="1.778" layer="95"/>
+</segment>
+<segment>
+<pinref part="AGND6" gate="VR1" pin="AGND"/>
+<pinref part="R16" gate="G$1" pin="1"/>
+<wire x1="-10.16" y1="-106.68" x2="-10.16" y2="-99.06" width="0.1524" layer="91"/>
+</segment>
+<segment>
+<pinref part="AGND8" gate="VR1" pin="AGND"/>
+<pinref part="C1" gate="G$1" pin="2"/>
+<wire x1="-50.8" y1="-106.68" x2="-50.8" y2="-83.82" width="0.1524" layer="91"/>
+</segment>
+<segment>
+<pinref part="C2" gate="G$1" pin="2"/>
+<pinref part="AGND7" gate="VR1" pin="AGND"/>
+<wire x1="-17.78" y1="-83.82" x2="-17.78" y2="-106.68" width="0.1524" layer="91"/>
 </segment>
 </net>
@@
 </segment>
 </net>
+<net name="N$14" class="0">
+<segment>
+<pinref part="C4" gate="G$1" pin="-"/>
+<pinref part="R13" gate="G$1" pin="1"/>
+<wire x1="-71.12" y1="-71.12" x2="-63.5" y2="-71.12" width="0.1524" layer="91"/>
+</segment>
+</net>
