File: powerSupply.sch (EAGLE design)
At the start: 19 parts, among them IC1 7915, IC2 7815TV

Commit message: блока питания продлжение
Parts:
- added C10: 0.1u, rcl:C-EUC0805
- added C11, C9: 220uF 10V, rcl:CPOL-EUUD-6,3X8,8
- added IC3: LM1117-5V, burr-brown:REG1117
- added IC4: LM317MABDT, v-reg:LM317MABDT
- added R6: 240, rcl:R-EU_M1206
- added R7: 5k, resistor:R-TRIMM3296W
Connections:
- net N$3 renamed +15V
- net N$4 renamed -15V
- removed net N$12: C1.+, L1.2, R4.1
- new net 3.6VADJ: C11.+, IC4.OUT, R6.1
- new net 5V: C9.+, IC3.VOUT
- new net 7V: C1.+, C10.2, IC3.VIN, IC4.IN, L1.2, R4.1
- new net N$5: B1.AC1
- new net N$6: B1.AC2
- new net N$8: IC4.ADJ, R6.2, R7.E, R7.S
- net AGND: now also C10.1, C11.-, C9.-, IC3.GND, R7.A
Changed lines of the file:
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@@
 <part name="AGND12" library="supply1" deviceset="AGND" device=""/>
 <part name="AGND13" library="supply1" deviceset="AGND" device=""/>
+<part name="IC3" library="burr-brown" deviceset="REG1117" device="" value="LM1117-5V"/>
+<part name="AGND14" library="supply1" deviceset="AGND" device=""/>
+<part name="C9" library="rcl" deviceset="CPOL-EU" device="UD-6,3X8,8" value="220uF 10V"/>
+<part name="AGND15" library="supply1" deviceset="AGND" device=""/>
+<part name="IC4" library="v-reg" deviceset="LM317?*" device="" technology="MABDT"/>
+<part name="C10" library="rcl" deviceset="C-EU" device="C0805" value="0.1u"/>
+<part name="R6" library="rcl" deviceset="R-EU_" device="M1206" value="240"/>
+<part name="R7" library="resistor" deviceset="R-TRIMM" device="3296W" value="5k"/>
+<part name="AGND16" library="supply1" deviceset="AGND" device=""/>
+<part name="C11" library="rcl" deviceset="CPOL-EU" device="UD-6,3X8,8" value="220uF 10V"/>
+<part name="AGND17" library="supply1" deviceset="AGND" device=""/>
+<part name="AGND18" library="supply1" deviceset="AGND" device=""/>
+<part name="AGND19" library="supply1" deviceset="AGND" device=""/>
 </parts>
 <sheets>
@@
 <instance part="AGND12" gate="VR1" x="60.96" y="25.4"/>
 <instance part="AGND13" gate="VR1" x="71.12" y="25.4"/>
+<instance part="IC3" gate="G$1" x="93.98" y="43.18"/>
+<instance part="AGND14" gate="VR1" x="93.98" y="25.4"/>
+<instance part="C9" gate="G$1" x="109.22" y="35.56"/>
+<instance part="AGND15" gate="VR1" x="109.22" y="25.4"/>
+<instance part="IC4" gate="G$1" x="104.14" y="91.44"/>
+<instance part="C10" gate="G$1" x="91.44" y="81.28" rot="R180"/>
+<instance part="R6" gate="G$1" x="127" y="83.82" rot="R270"/>
+<instance part="R7" gate="G$1" x="104.14" y="68.58"/>
+<instance part="AGND16" gate="VR1" x="104.14" y="58.42"/>
+<instance part="C11" gate="G$1" x="137.16" y="76.2"/>
+<instance part="AGND17" gate="VR1" x="137.16" y="58.42"/>
+<instance part="AGND18" gate="VR1" x="91.44" y="58.42"/>
+<instance part="AGND19" gate="VR1" x="-63.5" y="-40.64"/>
 </instances>
 <busses>
@@
 <wire x1="71.12" y1="27.94" x2="71.12" y2="30.48" width="0.1524" layer="91"/>
 </segment>
-</net>
-<net name="N$3" class="0">
+<segment>
+<pinref part="AGND14" gate="VR1" pin="AGND"/>
+<pinref part="IC3" gate="G$1" pin="GND"/>
+<wire x1="93.98" y1="27.94" x2="93.98" y2="30.48" width="0.1524" layer="91"/>
+</segment>
+<segment>
+<pinref part="AGND15" gate="VR1" pin="AGND"/>
+<pinref part="C9" gate="G$1" pin="-"/>
+<wire x1="109.22" y1="27.94" x2="109.22" y2="30.48" width="0.1524" layer="91"/>
+</segment>
+<segment>
+<pinref part="R7" gate="G$1" pin="A"/>
+<pinref part="AGND16" gate="VR1" pin="AGND"/>
+<wire x1="104.14" y1="63.5" x2="104.14" y2="60.96" width="0.1524" layer="91"/>
+</segment>
+<segment>
+<pinref part="C11" gate="G$1" pin="-"/>
+<pinref part="AGND17" gate="VR1" pin="AGND"/>
+<wire x1="137.16" y1="71.12" x2="137.16" y2="60.96" width="0.1524" layer="91"/>
+</segment>
+<segment>
+<pinref part="AGND18" gate="VR1" pin="AGND"/>
+<pinref part="C10" gate="G$1" pin="1"/>
+<wire x1="91.44" y1="60.96" x2="91.44" y2="78.74" width="0.1524" layer="91"/>
+</segment>
+<segment>
+<pinref part="AGND19" gate="VR1" pin="AGND"/>
+<wire x1="-63.5" y1="-38.1" x2="-63.5" y2="-12.7" width="0.1524" layer="91"/>
+<wire x1="-63.5" y1="-12.7" x2="-76.2" y2="-12.7" width="0.1524" layer="91"/>
+</segment>
+</net>
+<net name="+15V" class="0">
 <segment>
 <pinref part="IC2" gate="A1" pin="VO"/>
@@
 <wire x1="25.4" y1="12.7" x2="33.02" y2="12.7" width="0.1524" layer="91"/>
 <wire x1="33.02" y1="12.7" x2="33.02" y2="7.62" width="0.1524" layer="91"/>
-</segment>
-</net>
-<net name="N$4" class="0">
+<wire x1="33.02" y1="12.7" x2="50.8" y2="12.7" width="0.1524" layer="91"/>
+<junction x="33.02" y="12.7"/>
+<label x="45.72" y="12.7" size="1.778" layer="95"/>
+</segment>
+</net>
+<net name="-15V" class="0">
 <segment>
 <pinref part="IC1" gate="A1" pin="VO"/>
@@
 <wire x1="25.4" y1="-22.86" x2="33.02" y2="-22.86" width="0.1524" layer="91"/>
 <wire x1="33.02" y1="-22.86" x2="33.02" y2="-27.94" width="0.1524" layer="91"/>
+<wire x1="33.02" y1="-22.86" x2="50.8" y2="-22.86" width="0.1524" layer="91"/>
+<junction x="33.02" y="-22.86"/>
+<label x="45.72" y="-22.86" size="1.778" layer="95"/>
 </segment>
 </net>
@@
 </segment>
 </net>
-<net name="N$12" class="0">
+<net name="7V" class="0">
 <segment>
 <pinref part="L1" gate="G$1" pin="2"/>
@@
 <wire x1="25.4" y1="43.18" x2="71.12" y2="43.18" width="0.1524" layer="91"/>
 <junction x="71.12" y="43.18"/>
+<pinref part="IC3" gate="G$1" pin="VIN"/>
+<wire x1="81.28" y1="43.18" x2="78.74" y2="43.18" width="0.1524" layer="91"/>
+<label x="76.2" y="43.18" size="1.778" layer="95"/>
+<pinref part="C10" gate="G$1" pin="2"/>
+<pinref part="IC4" gate="G$1" pin="IN"/>
+<wire x1="78.74" y1="43.18" x2="71.12" y2="43.18" width="0.1524" layer="91"/>
+<wire x1="91.44" y1="86.36" x2="91.44" y2="91.44" width="0.1524" layer="91"/>
+<wire x1="91.44" y1="91.44" x2="96.52" y2="91.44" width="0.1524" layer="91"/>
+<wire x1="91.44" y1="91.44" x2="78.74" y2="91.44" width="0.1524" layer="91"/>
+<wire x1="78.74" y1="91.44" x2="78.74" y2="43.18" width="0.1524" layer="91"/>
+<junction x="91.44" y="91.44"/>
+<junction x="78.74" y="43.18"/>
 </segment>
 </net>
@@
 </segment>
 </net>
+<net name="5V" class="0">
+<segment>
+<pinref part="IC3" gate="G$1" pin="VOUT"/>
+<pinref part="C9" gate="G$1" pin="+"/>
+<wire x1="106.68" y1="43.18" x2="109.22" y2="43.18" width="0.1524" layer="91"/>
+<wire x1="109.22" y1="43.18" x2="109.22" y2="38.1" width="0.1524" layer="91"/>
+<label x="121.92" y="43.18" size="1.778" layer="95"/>
+<wire x1="109.22" y1="43.18" x2="124.46" y2="43.18" width="0.1524" layer="91"/>
+<junction x="109.22" y="43.18"/>
+</segment>
+</net>
+<net name="3.6VADJ" class="0">
+<segment>
+<pinref part="IC4" gate="G$1" pin="OUT"/>
+<pinref part="R6" gate="G$1" pin="1"/>
+<wire x1="111.76" y1="91.44" x2="127" y2="91.44" width="0.1524" layer="91"/>
+<wire x1="127" y1="91.44" x2="127" y2="88.9" width="0.1524" layer="91"/>
+<pinref part="C11" gate="G$1" pin="+"/>
+<wire x1="127" y1="91.44" x2="137.16" y2="91.44" width="0.1524" layer="91"/>
+<wire x1="137.16" y1="91.44" x2="137.16" y2="78.74" width="0.1524" layer="91"/>
+<junction x="127" y="91.44"/>
+<wire x1="137.16" y1="91.44" x2="152.4" y2="91.44" width="0.1524" layer="91"/>
+<junction x="137.16" y="91.44"/>
+<label x="142.24" y="91.44" size="1.778" layer="95"/>
+</segment>
+</net>
+<net name="N$8" class="0">
+<segment>
+<pinref part="R7" gate="G$1" pin="E"/>
+<pinref part="IC4" gate="G$1" pin="ADJ"/>
+<wire x1="104.14" y1="83.82" x2="104.14" y2="76.2" width="0.1524" layer="91"/>
+<wire x1="104.14" y1="76.2" x2="111.76" y2="76.2" width="0.1524" layer="91"/>
+<pinref part="R6" gate="G$1" pin="2"/>
+<wire x1="111.76" y1="76.2" x2="127" y2="76.2" width="0.1524" layer="91"/>
+<wire x1="127" y1="76.2" x2="127" y2="78.74" width="0.1524" layer="91"/>
+<wire x1="104.14" y1="73.66" x2="104.14" y2="76.2" width="0.1524" layer="91"/>
+<junction x="104.14" y="76.2"/>
+<pinref part="R7" gate="G$1" pin="S"/>
+<wire x1="109.22" y1="68.58" x2="111.76" y2="68.58" width="0.1524" layer="91"/>
+<wire x1="111.76" y1="68.58" x2="111.76" y2="76.2" width="0.1524" layer="91"/>
+<junction x="111.76" y="76.2"/>
+</segment>
+</net>
+<net name="N$5" class="0">
+<segment>
+<pinref part="B1" gate="1" pin="AC1"/>
+<wire x1="-33.02" y1="-7.62" x2="-76.2" y2="-7.62" width="0.1524" layer="91"/>
+</segment>
+</net>
+<net name="N$6" class="0">
+<segment>
+<pinref part="B1" gate="1" pin="AC2"/>
+<wire x1="-22.86" y1="-7.62" x2="-22.86" y2="-17.78" width="0.1524" layer="91"/>
+<wire x1="-22.86" y1="-17.78" x2="-76.2" y2="-17.78" width="0.1524" layer="91"/>
+</segment>
+</net>
